Commit message: docker

File: simulation/rom2109_description/urdf/rom2109_tall.xacro (robot description, xacro)
@@ -1,9 +1,11 @@
-<?xml version="1.0" encoding="utf-8"?>
-<!-- This URDF was automatically created by SolidWorks to URDF Exporter! Originally created by Stephen Brawner (brawner@gmail.com)
-     Commit Version: 1.6.0-1-g15f4949  Build Version: 1.6.7594.29634
-     For more information, please see http://wiki.ros.org/sw_urdf_exporter -->
-<robot
-  name="rom2109">
-  <link
+<?xml version="1.0"?>
+<robot xmlns:xacro="http://www.ros.org/wiki/xacro">
+    <link name="base_footprint"></link>
+    <joint name="base_footprint_joint" type="fixed">
+      <parent link="base_footprint"/>
+      <child link="base_link"/>
+      <origin xyz="0 0 0" rpy="0 0 0"/>
+    </joint>
+    <link
     name="base_link">
     <inertial>
@@ -416,44 +418,11 @@
       xyz="0 0 0" />
   </joint>
-    <!--GAZEBO ADD BY ROM ROBOTICS-->
-  <!-- here is the gazebo plug-in to simulate a lidar sensor -->
-  <gazebo reference="lidar">
-    <sensor type="ray" name="head_hokuyo_sensor">
-    <!--sensor type="gpu_ray" name="sick_lidar_sensor"-->
-      <pose>0 0 0 0 0 0</pose>
-      <visualize>true</visualize>
-      <update_rate>40</update_rate>
-      <ray>
-        <scan>
-          <horizontal>
-            <samples>720</samples>
-            <resolution>1</resolution>
-            <min_angle>-1.570796</min_angle>
-            <max_angle>1.570796</max_angle>
-          </horizontal>
-        </scan>
-        <range>
-          <min>0.10</min>
-          <max>30.0</max>
-          <resolution>0.01</resolution>
-        </range>
-        <noise>
-          <type>gaussian</type>
-          <mean>0.0</mean>
-          <stddev>0.01</stddev>
-        </noise>
-      </ray>
-      <!--plugin name="gazebo_ros_lidar_controller" filename="libgazebo_ros_gpu_laser.so"-->
-      <plugin name="gazebo_ros_head_hokuyo_controller" filename="libgazebo_ros_laser.so">
-        <topicName>/scan</topicName>
-        <frameName>lidar</frameName>
-      </plugin>
-    </sensor>
-  </gazebo>
-<gazebo>
-  <plugin name="gazebo_ros_control" filename="libgazebo_ros_contol.so">
-  </plugin>
-</gazebo>
- <!-- Colour -->
+    <link name="imu_link"/>
+    <joint name="imu_joint" type="fixed">
+      <parent link="base_link"/>
+      <child link="imu_link"/>
+      <origin rpy="0 0 0" xyz="0 0 0"/>
+    </joint>
+  <!-- Colour -->
   <gazebo reference="base_link">
     <material>Gazebo/Black</material>
@@ -468,21 +437,3 @@
     <material>Gazebo/Yellow</material>
   </gazebo>
-  <gazebo>
-    <plugin name="differential_drive_controller" filename="libgazebo_ros_diff_drive.so">
-      <alwaysOn>true</alwaysOn>
-	    <updateRate>10.0</updateRate>
-		  <robotBaseFrame>base_link</robotBaseFrame>
-		  <publishWheelTF>true</publishWheelTF>
-		  <publishWheelJointState>true</publishWheelJointState>
-		  <wheelAcceleration>1</wheelAcceleration>
-		  <leftJoint>left_wheel_joint</leftJoint>
-		  <rightJoint>right_wheel_joint</rightJoint>
-		  <wheelSeparation>0.33</wheelSeparation>
-		  <wheelDiameter>0.17</wheelDiameter>
-		  <wheelTorque>20</wheelTorque>
-		  <commandTopic>cmd_vel</commandTopic>
-		  <odometryTopic>odom</odometryTopic>
-		  <odometryFrame>odom</odometryFrame>
-    </plugin>
- </gazebo>
 </robot>
